File: Hardware/RoomBouy/RoomBouy.kicad_pcb (KiCad board)
At the start: 2 copper layers, 65 x 56.5 mm, 38 parts, among them J1 Roomba Wake, J2 Raspberry_Pi_2_3, J3 Roomba Connector, J4 ProtoPad, J5 Servo, Q1 MMBT3904, Q2 MMBT3904, Q3 MMBT3906, Q4 MMBT3904, Q5 2SB772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

Commit message: rename txd thru all
Parts:
- D1: value TXD -> RXD
- D2: value RXD -> TXD
Connections:
- D1 pad 2: /ROOMBA_TXD -> /ROOMBA_RXD
- D2 pad 2: /ROOMBA_RXD -> /ROOMBA_TXD
- J3 pad 2: /ROOMBA_RXD -> /ROOMBA_TXD
- J3 pad 3: /ROOMBA_TXD -> /ROOMBA_RXD
- R2 pad 1: /ROOMBA_TXD -> /ROOMBA_RXD
- R6 pad 2: /ROOMBA_RXD -> /ROOMBA_TXD
Routing:
- net /ROOMBA_TXD: track 39.8 -> 43.3 mm, vias 2 -> 0
- net /ROOMBA_RXD: track 43.3 -> 39.8 mm, vias 0 -> 2
