File: Hardware/RoomBouy/RoomBouy.kicad_sch (KiCad schematic)
At the start: 34 parts, among them J1 Roomba Wake, J2 Raspberry_Pi_2_3, J3 Roomba Connector, J4 ProtoPad, J5 Servo, Q1 MMBT3904, Q2 MMBT3904, Q3 MMBT3906, Q4 MMBT3904, Q5 2SB772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

Commit message: rename txd thru all
Parts:
- D1: value TXD -> RXD
- D2: value RXD -> TXD
Connections:
- net ROOMBA_RXD: now also D1.2 (A), J3.3 (Pin_3), R2.1; no longer D2.2 (A), J3.2 (Pin_2), R6.2
- net ROOMBA_TXD: now also D2.2 (A), J3.2 (Pin_2), R6.2; no longer D1.2 (A), J3.3 (Pin_3), R2.1
Changed lines of the file:
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@@
 		)
 	)
-	(label "ROOMBA_TXD"
+	(label "ROOMBA_RXD"
 		(at 77.47 38.1 0)
 		(effects
@@
 		)
 	)
-	(label "ROOMBA_RXD"
+	(label "ROOMBA_TXD"
 		(at 60.96 31.75 180)
 		(effects
@@
 		)
 	)
-	(label "ROOMBA_TXD"
+	(label "ROOMBA_RXD"
 		(at 165.1 22.86 0)
 		(effects
@@
 		)
 	)
-	(label "ROOMBA_RXD"
+	(label "ROOMBA_TXD"
 		(at 165.1 34.29 0)
 		(effects
@@
 		)
 	)
-	(label "ROOMBA_TXD"
+	(label "ROOMBA_RXD"
 		(at 60.96 29.21 180)
 		(effects
@@
 		)
 	)
-	(label "ROOMBA_RXD"
+	(label "ROOMBA_TXD"
 		(at 158.75 63.5 180)
 		(effects
@@
 			)
 		)
-		(property "Value" "RXD"
+		(property "Value" "TXD"
 			(at 184.4675 29.21 0)
 			(effects
@@
 			)
 		)
-		(property "Value" "TXD"
+		(property "Value" "RXD"
 			(at 184.4675 17.78 0)
 			(effects
